File: Space Cowboy RBG.sch (KiCad schematic (older format))
At the start: 32 parts

Commit message: Update Space Cowboy RBG.sch
Parts:
- added CRGB17, CRGB18: 0.1uF, symbol Device:C_Small
- added DRGB17, DRGB18: WS2812B, LED_SMD:LED_WS2812B_PLCC4_5.0x5.0mm_P3.2mm, symbol LED:WS2812B
Connections:
- net +5V: now also CRGB17.1, CRGB18.1, DRGB17.1 (VDD), DRGB18.1 (VDD)
- net GND: now also CRGB17.2, CRGB18.2, DRGB17.3 (VSS), DRGB18.3 (VSS)
- net at DRGB16.2 (DOUT): now also DRGB17.4 (DIN)
- new net: DRGB17.2 (DOUT), DRGB18.4 (DIN)
Changed lines of the file:
@@
 Wire Wire Line
 	3900 6750 4350 6750
-NoConn ~ 3600 1200
 $Comp
 L Device:C_Small CRGB1
@@
 Connection ~ 9400 4600
 Wire Wire Line
-	9400 4600 10650 4600
+	9400 4600 9800 4600
 Wire Wire Line
 	9800 3800 10200 3800
@@
 Text GLabel 5750 7050 3    50   Input ~ 0
 RGB_DI_PIN
+$Comp
+L LED:WS2812B DRGB17
+U 1 1 5FED22E9
+P 1450 6750
+F 0 "DRGB17" V 1496 6406 50  0000 R CNN
+F 1 "WS2812B" V 1405 6406 50  0000 R CNN
+F 2 "LED_SMD:LED_WS2812B_PLCC4_5.0x5.0mm_P3.2mm" H 1500 6450 50  0001 L TNN
+F 3 "https://cdn-shop.adafruit.com/datasheets/WS2812B.pdf" H 1550 6375 50  0001 L TNN
+	1    1450 6750
+	0    -1   -1   0
+$EndComp
+$Comp
+L power:+5V #PWR?
+U 1 1 5FED22EF
+P 1000 6750
+F 0 "#PWR?" H 1000 6600 50  0001 C CNN
+F 1 "+5V" H 1015 6923 50  0000 C CNN
+F 2 "" H 1000 6750 50  0001 C CNN
+F 3 "" H 1000 6750 50  0001 C CNN
+	1    1000 6750
+	1    0    0    -1
+$EndComp
+$Comp
+L power:GND #PWR?
+U 1 1 5FED22F5
+P 2200 6750
+F 0 "#PWR?" H 2200 6500 50  0001 C CNN
+F 1 "GND" H 2205 6577 50  0000 C CNN
+F 2 "" H 2200 6750 50  0001 C CNN
+F 3 "" H 2200 6750 50  0001 C CNN
+	1    2200 6750
+	1    0    0    -1
+$EndComp
+Wire Wire Line
+	1000 6750 1150 6750
+Wire Wire Line
+	1750 6750 2200 6750
+$Comp
+L LED:WS2812B DRGB18
+U 1 1 5FED80EC
+P 1450 6000
+F 0 "DRGB18" V 1496 5656 50  0000 R CNN
+F 1 "WS2812B" V 1405 5656 50  0000 R CNN
+F 2 "LED_SMD:LED_WS2812B_PLCC4_5.0x5.0mm_P3.2mm" H 1500 5700 50  0001 L TNN
+F 3 "https://cdn-shop.adafruit.com/datasheets/WS2812B.pdf" H 1550 5625 50  0001 L TNN
+	1    1450 6000
+	0    -1   -1   0
+$EndComp
+$Comp
+L power:+5V #PWR?
+U 1 1 5FED80F2
+P 1000 6000
+F 0 "#PWR?" H 1000 5850 50  0001 C CNN
+F 1 "+5V" H 1015 6173 50  0000 C CNN
+F 2 "" H 1000 6000 50  0001 C CNN
+F 3 "" H 1000 6000 50  0001 C CNN
+	1    1000 6000
+	1    0    0    -1
+$EndComp
+$Comp
+L power:GND #PWR?
+U 1 1 5FED80F8
+P 2200 6000
+F 0 "#PWR?" H 2200 5750 50  0001 C CNN
+F 1 "GND" H 2205 5827 50  0000 C CNN
+F 2 "" H 2200 6000 50  0001 C CNN
+F 3 "" H 2200 6000 50  0001 C CNN
+	1    2200 6000
+	1    0    0    -1
+$EndComp
+Wire Wire Line
+	1000 6000 1150 6000
+Wire Wire Line
+	1750 6000 2200 6000
+NoConn ~ 1450 5700
+$Comp
+L Device:C_Small CRGB17
+U 1 1 5FEE09D6
+P 9800 4500
+F 0 "CRGB17" H 9892 4546 50  0000 L CNN
+F 1 "0.1uF" H 9892 4455 50  0000 L CNN
+F 2 "" H 9800 4500 50  0001 C CNN
+F 3 "~" H 9800 4500 50  0001 C CNN
+	1    9800 4500
+	1    0    0    -1
+$EndComp
+Connection ~ 9800 4600
+Wire Wire Line
+	9800 4600 10200 4600
+$Comp
+L Device:C_Small CRGB18
+U 1 1 5FEE161A
+P 10200 4500
+F 0 "CRGB18" H 10292 4546 50  0000 L CNN
+F 1 "0.1uF" H 10292 4455 50  0000 L CNN
+F 2 "" H 10200 4500 50  0001 C CNN
+F 3 "~" H 10200 4500 50  0001 C CNN
+	1    10200 4500
+	1    0    0    -1
+$EndComp
+Connection ~ 10200 4600
+Wire Wire Line
+	10200 4600 10650 4600
+Wire Wire Line
+	9400 4400 9800 4400
+Connection ~ 9400 4400
+Connection ~ 9800 4400
+Wire Wire Line
+	9800 4400 10200 4400
+Wire Wire Line
+	1450 7250 2750 7250
+Wire Wire Line
+	2750 7250 2750 950
+Wire Wire Line
+	2750 950  3600 950
+Wire Wire Line
+	3600 950  3600 1200
+Wire Wire Line
+	1450 7050 1450 7250
+Wire Wire Line
+	1450 6300 1450 6450
 $EndSCHEMATC

Commit message: Update Space Cowboy RBG.sch
Parts:
- CRGB1, CRGB10, CRGB11, CRGB12, CRGB13, CRGB14, CRGB15, CRGB16, CRGB17, CRGB18, CRGB2, CRGB3, CRGB4, CRGB5, CRGB6, CRGB7, CRGB8, CRGB9: footprint (none) -> Capacitors_SMD:C_0603
- DRGB1, DRGB10, DRGB11, DRGB12, DRGB13, DRGB14, DRGB15, DRGB16, DRGB17, DRGB18, DRGB2, DRGB3, DRGB4, DRGB5, DRGB6, DRGB7, DRGB8, DRGB9: footprint LED_SMD:LED_WS2812B_PLCC4_5.0x5.0mm_P3.2mm -> WS2812B Worldsemi:WS2812B
