File: Space Cowboy RBG.sch (KiCad schematic (older format))
At the start: 36 parts

Commit message: Update Space Cowboy RBG.sch
Parts:
- DRGB1, DRGB10, DRGB11, DRGB12, DRGB13, DRGB14, DRGB15, DRGB16, DRGB17, DRGB18, DRGB2, DRGB3, DRGB4, DRGB5, DRGB6, DRGB7, DRGB8, DRGB9: LCSC (none) -> C114586
Connections:
- net at DRGB18.2 (DOUT): now also DRGB1.4 (DIN)
Changed lines of the file:
@@
 F 2 "WS2812B Worldsemi:WS2812B" H 5800 6150 50  0001 L TNN
 F 3 "https://cdn-shop.adafruit.com/datasheets/WS2812B.pdf" H 5850 6075 50  0001 L TNN
+F 4 "C114586" V 5750 6450 50  0001 C CNN "LCSC"
 	1    5750 6450
 	0    -1   -1   0
@@
 F 2 "WS2812B Worldsemi:WS2812B" H 5800 5400 50  0001 L TNN
 F 3 "https://cdn-shop.adafruit.com/datasheets/WS2812B.pdf" H 5850 5325 50  0001 L TNN
+F 4 "C114586" V 5750 5700 50  0001 C CNN "LCSC"
 	1    5750 5700
 	0    -1   -1   0
@@
 F 2 "WS2812B Worldsemi:WS2812B" H 5800 4650 50  0001 L TNN
 F 3 "https://cdn-shop.adafruit.com/datasheets/WS2812B.pdf" H 5850 4575 50  0001 L TNN
+F 4 "C114586" V 5750 4950 50  0001 C CNN "LCSC"
 	1    5750 4950
 	0    -1   -1   0
@@
 F 2 "WS2812B Worldsemi:WS2812B" H 5800 3900 50  0001 L TNN
 F 3 "https://cdn-shop.adafruit.com/datasheets/WS2812B.pdf" H 5850 3825 50  0001 L TNN
+F 4 "C114586" V 5750 4200 50  0001 C CNN "LCSC"
 	1    5750 4200
 	0    -1   -1   0
@@
 F 2 "WS2812B Worldsemi:WS2812B" H 5800 3150 50  0001 L TNN
 F 3 "https://cdn-shop.adafruit.com/datasheets/WS2812B.pdf" H 5850 3075 50  0001 L TNN
+F 4 "C114586" V 5750 3450 50  0001 C CNN "LCSC"
 	1    5750 3450
 	0    -1   -1   0
@@
 F 2 "WS2812B Worldsemi:WS2812B" H 5800 2400 50  0001 L TNN
 F 3 "https://cdn-shop.adafruit.com/datasheets/WS2812B.pdf" H 5850 2325 50  0001 L TNN
+F 4 "C114586" V 5750 2700 50  0001 C CNN "LCSC"
 	1    5750 2700
 	0    -1   -1   0
@@
 F 2 "WS2812B Worldsemi:WS2812B" H 5800 1650 50  0001 L TNN
 F 3 "https://cdn-shop.adafruit.com/datasheets/WS2812B.pdf" H 5850 1575 50  0001 L TNN
+F 4 "C114586" V 5750 1950 50  0001 C CNN "LCSC"
 	1    5750 1950
 	0    -1   -1   0
@@
 F 2 "WS2812B Worldsemi:WS2812B" H 5800 900 50  0001 L TNN
 F 3 "https://cdn-shop.adafruit.com/datasheets/WS2812B.pdf" H 5850 825 50  0001 L TNN
+F 4 "C114586" V 5750 1200 50  0001 C CNN "LCSC"
 	1    5750 1200
 	0    -1   -1   0
@@
 F 2 "WS2812B Worldsemi:WS2812B" H 3650 6150 50  0001 L TNN
 F 3 "https://cdn-shop.adafruit.com/datasheets/WS2812B.pdf" H 3700 6075 50  0001 L TNN
+F 4 "C114586" V 3600 6450 50  0001 C CNN "LCSC"
 	1    3600 6450
 	0    -1   -1   0
@@
 F 2 "WS2812B Worldsemi:WS2812B" H 3650 5400 50  0001 L TNN
 F 3 "https://cdn-shop.adafruit.com/datasheets/WS2812B.pdf" H 3700 5325 50  0001 L TNN
+F 4 "C114586" V 3600 5700 50  0001 C CNN "LCSC"
 	1    3600 5700
 	0    -1   -1   0
@@
 F 2 "WS2812B Worldsemi:WS2812B" H 3650 4650 50  0001 L TNN
 F 3 "https://cdn-shop.adafruit.com/datasheets/WS2812B.pdf" H 3700 4575 50  0001 L TNN
+F 4 "C114586" V 3600 4950 50  0001 C CNN "LCSC"
 	1    3600 4950
 	0    -1   -1   0
@@
 F 2 "WS2812B Worldsemi:WS2812B" H 3650 3900 50  0001 L TNN
 F 3 "https://cdn-shop.adafruit.com/datasheets/WS2812B.pdf" H 3700 3825 50  0001 L TNN
+F 4 "C114586" V 3600 4200 50  0001 C CNN "LCSC"
 	1    3600 4200
 	0    -1   -1   0
@@
 F 2 "WS2812B Worldsemi:WS2812B" H 3650 3150 50  0001 L TNN
 F 3 "https://cdn-shop.adafruit.com/datasheets/WS2812B.pdf" H 3700 3075 50  0001 L TNN
+F 4 "C114586" V 3600 3450 50  0001 C CNN "LCSC"
 	1    3600 3450
 	0    -1   -1   0
@@
 F 2 "WS2812B Worldsemi:WS2812B" H 3650 2400 50  0001 L TNN
 F 3 "https://cdn-shop.adafruit.com/datasheets/WS2812B.pdf" H 3700 2325 50  0001 L TNN
+F 4 "C114586" V 3600 2700 50  0001 C CNN "LCSC"
 	1    3600 2700
 	0    -1   -1   0
@@
 F 2 "WS2812B Worldsemi:WS2812B" H 3650 1650 50  0001 L TNN
 F 3 "https://cdn-shop.adafruit.com/datasheets/WS2812B.pdf" H 3700 1575 50  0001 L TNN
+F 4 "C114586" V 3600 1950 50  0001 C CNN "LCSC"
 	1    3600 1950
 	0    -1   -1   0
@@
 F 2 "WS2812B Worldsemi:WS2812B" H 3650 900 50  0001 L TNN
 F 3 "https://cdn-shop.adafruit.com/datasheets/WS2812B.pdf" H 3700 825 50  0001 L TNN
+F 4 "C114586" V 3600 1200 50  0001 C CNN "LCSC"
 	1    3600 1200
 	0    -1   -1   0
@@
 F 2 "WS2812B Worldsemi:WS2812B" H 1500 6150 50  0001 L TNN
 F 3 "https://cdn-shop.adafruit.com/datasheets/WS2812B.pdf" H 1550 6075 50  0001 L TNN
+F 4 "C114586" V 1450 6450 50  0001 C CNN "LCSC"
 	1    1450 6450
 	0    -1   -1   0
@@
 F 2 "WS2812B Worldsemi:WS2812B" H 5800 6900 50  0001 L TNN
 F 3 "https://cdn-shop.adafruit.com/datasheets/WS2812B.pdf" H 5850 6825 50  0001 L TNN
+F 4 "C114586" V 5750 7200 50  0001 C CNN "LCSC"
 	1    5750 7200
 	0    -1   -1   0
@@
 Wire Wire Line
 	1450 6000 1450 6150
+Wire Wire Line
+	5750 6750 5750 6900
 $EndSCHEMATC

Commit message: Update Space Cowboy RBG.sch
Parts:
- CRGB1, CRGB10, CRGB11, CRGB12, CRGB13, CRGB14, CRGB15, CRGB16, CRGB17, CRGB18, CRGB2, CRGB3, CRGB4, CRGB5, CRGB6, CRGB7, CRGB8, CRGB9: LCSC (none) -> C24452
Changed lines of the file:
@@
 F 2 "Capacitors_SMD:C_0603" H 8200 3700 50  0001 C CNN
 F 3 "~" H 8200 3700 50  0001 C CNN
+F 4 "C24452" H 8200 3700 50  0001 C CNN "LCSC"
 	1    8200 3700
 	1    0    0    -1
@@
 F 2 "Capacitors_SMD:C_0603" H 8600 3700 50  0001 C CNN
 F 3 "~" H 8600 3700 50  0001 C CNN
+F 4 "C24452" H 8600 3700 50  0001 C CNN "LCSC"
 	1    8600 3700
 	1    0    0    -1
@@
 F 2 "Capacitors_SMD:C_0603" H 9000 3700 50  0001 C CNN
 F 3 "~" H 9000 3700 50  0001 C CNN
+F 4 "C24452" H 9000 3700 50  0001 C CNN "LCSC"
 	1    9000 3700
 	1    0    0    -1
@@
 F 2 "Capacitors_SMD:C_0603" H 9400 3700 50  0001 C CNN
 F 3 "~" H 9400 3700 50  0001 C CNN
+F 4 "C24452" H 9400 3700 50  0001 C CNN "LCSC"
 	1    9400 3700
 	1    0    0    -1
@@
 F 2 "Capacitors_SMD:C_0603" H 9800 3700 50  0001 C CNN
 F 3 "~" H 9800 3700 50  0001 C CNN
+F 4 "C24452" H 9800 3700 50  0001 C CNN "LCSC"
 	1    9800 3700
 	1    0    0    -1
@@
 F 2 "Capacitors_SMD:C_0603" H 10200 3700 50  0001 C CNN
 F 3 "~" H 10200 3700 50  0001 C CNN
+F 4 "C24452" H 10200 3700 50  0001 C CNN "LCSC"
 	1    10200 3700
 	1    0    0    -1
@@
 F 2 "Capacitors_SMD:C_0603" H 8200 4100 50  0001 C CNN
 F 3 "~" H 8200 4100 50  0001 C CNN
+F 4 "C24452" H 8200 4100 50  0001 C CNN "LCSC"
 	1    8200 4100
 	1    0    0    -1
@@
 F 2 "Capacitors_SMD:C_0603" H 8600 4100 50  0001 C CNN
 F 3 "~" H 8600 4100 50  0001 C CNN
+F 4 "C24452" H 8600 4100 50  0001 C CNN "LCSC"
 	1    8600 4100
 	1    0    0    -1
@@
 F 2 "Capacitors_SMD:C_0603" H 9000 4100 50  0001 C CNN
 F 3 "~" H 9000 4100 50  0001 C CNN
+F 4 "C24452" H 9000 4100 50  0001 C CNN "LCSC"
 	1    9000 4100
 	1    0    0    -1
@@
 F 2 "Capacitors_SMD:C_0603" H 9400 4100 50  0001 C CNN
 F 3 "~" H 9400 4100 50  0001 C CNN
+F 4 "C24452" H 9400 4100 50  0001 C CNN "LCSC"
 	1    9400 4100
 	1    0    0    -1
@@
 F 2 "Capacitors_SMD:C_0603" H 9800 4100 50  0001 C CNN
 F 3 "~" H 9800 4100 50  0001 C CNN
+F 4 "C24452" H 9800 4100 50  0001 C CNN "LCSC"
 	1    9800 4100
 	1    0    0    -1
@@
 F 2 "Capacitors_SMD:C_0603" H 10200 4100 50  0001 C CNN
 F 3 "~" H 10200 4100 50  0001 C CNN
+F 4 "C24452" H 10200 4100 50  0001 C CNN "LCSC"
 	1    10200 4100
 	1    0    0    -1
@@
 F 2 "Capacitors_SMD:C_0603" H 8200 4500 50  0001 C CNN
 F 3 "~" H 8200 4500 50  0001 C CNN
+F 4 "C24452" H 8200 4500 50  0001 C CNN "LCSC"
 	1    8200 4500
 	1    0    0    -1
@@
 F 2 "Capacitors_SMD:C_0603" H 8600 4500 50  0001 C CNN
 F 3 "~" H 8600 4500 50  0001 C CNN
+F 4 "C24452" H 8600 4500 50  0001 C CNN "LCSC"
 	1    8600 4500
 	1    0    0    -1
@@
 F 2 "Capacitors_SMD:C_0603" H 9000 4500 50  0001 C CNN
 F 3 "~" H 9000 4500 50  0001 C CNN
+F 4 "C24452" H 9000 4500 50  0001 C CNN "LCSC"
 	1    9000 4500
 	1    0    0    -1
@@
 F 2 "Capacitors_SMD:C_0603" H 9400 4500 50  0001 C CNN
 F 3 "~" H 9400 4500 50  0001 C CNN
+F 4 "C24452" H 9400 4500 50  0001 C CNN "LCSC"
 	1    9400 4500
 	1    0    0    -1
@@
 F 2 "Capacitors_SMD:C_0603" H 9800 4500 50  0001 C CNN
 F 3 "~" H 9800 4500 50  0001 C CNN
+F 4 "C24452" H 9800 4500 50  0001 C CNN "LCSC"
 	1    9800 4500
 	1    0    0    -1
@@
 F 2 "Capacitors_SMD:C_0603" H 10200 4500 50  0001 C CNN
 F 3 "~" H 10200 4500 50  0001 C CNN
+F 4 "C24452" H 10200 4500 50  0001 C CNN "LCSC"
 	1    10200 4500
 	1    0    0    -1
